File: blinkey.sch (KiCad schematic (older format))
At the start: 5 parts, among them SW1 SW_Push, SW2 SW_Push, SW3 SW_Push, SW4 SW_Push, SW5 SW_Push

Commit message: LEDs
Parts:
- added D0, D1, D2, D3, D4, D5, D6, D7, D8: RED, LEDs:LED_0805, symbol LED_ALT
Connections:
- new net GND: D0.1 (K), D1.1 (K), D2.1 (K), D3.1 (K), D4.1 (K), D5.1 (K), D6.1 (K), D7.1 (K)
Changed lines of the file:
@@
 	1    0    0    -1
 $EndComp
+$Comp
+L LED_ALT D1
+U 1 1 5A12D865
+P 5000 2350
+F 0 "D1" H 5000 2250 50  0000 C CNN
+F 1 "RED" H 5300 2250 50  0000 C CNN
+F 2 "LEDs:LED_0805" H 5000 2350 50  0001 C CNN
+F 3 "" H 5000 2350 50  0001 C CNN
+	1    5000 2350
+	1    0    0    -1
+$EndComp
+$Comp
+L LED_ALT D2
+U 1 1 5A12D98A
+P 5000 2150
+F 0 "D2" H 5000 2050 50  0000 C CNN
+F 1 "RED" H 5300 2050 50  0000 C CNN
+F 2 "LEDs:LED_0805" H 5000 2150 50  0001 C CNN
+F 3 "" H 5000 2150 50  0001 C CNN
+	1    5000 2150
+	1    0    0    -1
+$EndComp
+$Comp
+L LED_ALT D3
+U 1 1 5A12D9E7
+P 5000 1950
+F 0 "D3" H 5000 1850 50  0000 C CNN
+F 1 "RED" H 5300 1850 50  0000 C CNN
+F 2 "LEDs:LED_0805" H 5000 1950 50  0001 C CNN
+F 3 "" H 5000 1950 50  0001 C CNN
+	1    5000 1950
+	1    0    0    -1
+$EndComp
+$Comp
+L LED_ALT D4
+U 1 1 5A12DA42
+P 3700 2550
+F 0 "D4" H 3700 2650 50  0000 C CNN
+F 1 "RED" H 3950 2650 50  0000 C CNN
+F 2 "LEDs:LED_0805" H 3700 2550 50  0001 C CNN
+F 3 "" H 3700 2550 50  0001 C CNN
+	1    3700 2550
+	-1   0    0    1
+$EndComp
+$Comp
+L LED_ALT D0
+U 1 1 5A12DECC
+P 5000 2550
+F 0 "D0" H 5000 2450 50  0000 C CNN
+F 1 "RED" H 5300 2450 50  0000 C CNN
+F 2 "LEDs:LED_0805" H 5000 2550 50  0001 C CNN
+F 3 "" H 5000 2550 50  0001 C CNN
+	1    5000 2550
+	1    0    0    -1
+$EndComp
+$Comp
+L LED_ALT D5
+U 1 1 5A12E5F5
+P 3700 2350
+F 0 "D5" H 3700 2450 50  0000 C CNN
+F 1 "RED" H 3950 2450 50  0000 C CNN
+F 2 "LEDs:LED_0805" H 3700 2350 50  0001 C CNN
+F 3 "" H 3700 2350 50  0001 C CNN
+	1    3700 2350
+	-1   0    0    1
+$EndComp
+$Comp
+L LED_ALT D6
+U 1 1 5A12E666
+P 3700 2150
+F 0 "D6" H 3700 2250 50  0000 C CNN
+F 1 "RED" H 3950 2250 50  0000 C CNN
+F 2 "LEDs:LED_0805" H 3700 2150 50  0001 C CNN
+F 3 "" H 3700 2150 50  0001 C CNN
+	1    3700 2150
+	-1   0    0    1
+$EndComp
+$Comp
+L LED_ALT D7
+U 1 1 5A12E729
+P 3700 1950
+F 0 "D7" H 3700 2050 50  0000 C CNN
+F 1 "RED" H 3950 2050 50  0000 C CNN
+F 2 "LEDs:LED_0805" H 3700 1950 50  0001 C CNN
+F 3 "" H 3700 1950 50  0001 C CNN
+	1    3700 1950
+	-1   0    0    1
+$EndComp
+Wire Wire Line
+	3850 1950 3900 1950
+Wire Wire Line
+	3900 1950 3900 2600
+Wire Wire Line
+	3850 2550 3900 2550
+Connection ~ 3900 2550
+Wire Wire Line
+	3850 2350 3900 2350
+Connection ~ 3900 2350
+Wire Wire Line
+	3850 2150 3900 2150
+Connection ~ 3900 2150
+$Comp
+L GND #PWR06
+U 1 1 5A12EBE6
+P 3900 2600
+F 0 "#PWR06" H 3900 2350 50  0001 C CNN
+F 1 "GND" H 3900 2450 50  0000 C CNN
+F 2 "" H 3900 2600 50  0001 C CNN
+F 3 "" H 3900 2600 50  0001 C CNN
+	1    3900 2600
+	1    0    0    -1
+$EndComp
+Wire Wire Line
+	4850 1950 4800 1950
+Wire Wire Line
+	4800 1950 4800 2600
+Wire Wire Line
+	4850 2550 4800 2550
+Connection ~ 4800 2550
+Wire Wire Line
+	4850 2350 4800 2350
+Connection ~ 4800 2350
+Wire Wire Line
+	4850 2150 4800 2150
+Connection ~ 4800 2150
+$Comp
+L GND #PWR07
+U 1 1 5A12EC81
+P 4800 2600
+F 0 "#PWR07" H 4800 2350 50  0001 C CNN
+F 1 "GND" H 4800 2450 50  0000 C CNN
+F 2 "" H 4800 2600 50  0001 C CNN
+F 3 "" H 4800 2600 50  0001 C CNN
+	1    4800 2600
+	1    0    0    -1
+$EndComp
+$Comp
+L LED_ALT D8
+U 1 1 5A12F069
+P 4350 1850
+F 0 "D8" H 4350 1950 50  0000 C CNN
+F 1 "RED" H 4600 1950 50  0000 C CNN
+F 2 "LEDs:LED_0805" H 4350 1850 50  0001 C CNN
+F 3 "" H 4350 1850 50  0001 C CNN
+	1    4350 1850
+	0    -1   -1   0
+$EndComp
 $EndSCHEMATC
