File: usb.sch (KiCad schematic (older format))
At the start: 4 parts, among them J4 USB_OTG, J5 Conn_01x06, U3 FT232RL, Y1 FNETHE025

Commit message: usbserial FT232RL changed to FT231XS
Parts:
- removed U3: FT232RL, Housings_SSOP:SSOP-28_5.3x10.2mm_Pitch0.65mm, symbol FT232RL
- added U3: FT231XS, SMD_Packages:SSOP-20, symbol FT231XS
Changed lines of the file:
@@
 JTAG_TDI
 $Comp
-L FT232RL U3
-U 1 1 5A1333CB
-P 5850 3000
-F 0 "U3" H 5200 3900 50  0000 L CNN
-F 1 "FT232RL" H 6250 3900 50  0000 L CNN
-F 2 "Housings_SSOP:SSOP-28_5.3x10.2mm_Pitch0.65mm" H 5850 3000 50  0001 C CNN
-F 3 "" H 5850 3000 50  0001 C CNN
-	1    5850 3000
+L FT231XS U3
+U 1 1 5A134DAE
+P 7850 3000
+F 0 "U3" H 7300 3800 50  0000 L CNN
+F 1 "FT231XS" H 8150 3800 50  0000 L CNN
+F 2 "SMD_Packages:SSOP-20" H 7850 3000 50  0001 C CNN
+F 3 "" H 7850 3000 50  0001 C CNN
+	1    7850 3000
 	1    0    0    -1
 $EndComp
