File: ulx2s.kicad_pcb (KiCad board)
At the start: 4 copper layers, 35.6 x 61 mm, 28 parts, among them J1 Conn_01x24, J2 Conn_01x24, J3 Micro_SD_Card_Det, J4 USB_OTG, J5 Conn_01x06, J6 Audio-Jack-5, P1 MICRO-HDMI-D, SW1 SW_Push, SW2 SW_Push, SW3 SW_Push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

Commit message: PCB: update after footprint and schem changes
Parts:
- J6: value Audio-Jack-5 -> JACK_TRS_6PINS
Changed lines of the file:
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@@
 (kicad_pcb (version 4) (host pcbnew 4.0.7+dfsg1-1)
   (general
-    (links 35)
-    (no_connects 35)
-    (area 131.464999 79.305 186.035001 151.745001)
+    (links 36)
+    (no_connects 36)
+    (area 140.894999 81.204999 176.605001 142.315001)
     (thickness 1.6)
     (drawings 4)
@@
     (zones 0)
     (modules 28)
-    (nets 13)
+    (nets 14)
   )
   (page A4)
@@
   (net 11 "Net-(SW5-Pad2)")
   (net 12 "Net-(SW5-Pad1)")
+  (net 13 "Net-(P1-Pad0)")
   (net_class Default "This is the default net class."
     (clearance 0.2)
@@
     (add_net +3V3)
     (add_net GND)
+    (add_net "Net-(P1-Pad0)")
     (add_net "Net-(SW1-Pad1)")
     (add_net "Net-(SW1-Pad2)")
@@
       (effects (font (size 0.6096 0.6096) (thickness 0.1524)) (justify mirror))
     )
-    (fp_text value Audio-Jack-5 (at 1.519498 -0.28335 270) (layer B.SilkS)
+    (fp_text value JACK_TRS_6PINS (at 1.519498 -0.28335 270) (layer B.SilkS)
       (effects (font (size 1 1) (thickness 0.15)) (justify mirror))
     )
@@
     (pad "" np_thru_hole circle (at 0 -4 270) (size 1.7 1.7) (drill 1.7) (layers *.Cu *.Mask B.SilkS)
       (clearance 0.4))
-  )
-  (module micro-hdmi-d:MICRO-HDMI-D (layer B.Cu)
-    (at 168.91 81.11)
-    (attr smd)
-    (fp_text reference P1 (at -0.025 3.125) (layer B.SilkS)
-      (effects (font (size 0.3 0.3) (thickness 0.075)) (justify mirror))
-    )
-    (fp_text value MICRO-HDMI-D (at 0 1.6) (layer B.SilkS)
-      (effects (font (size 0.3 0.3) (thickness 0.075)) (justify mirror))
-    )
-    (fp_line (start -3.3 0) (end -3.3 -0.7) (layer B.SilkS) (width 0.001))
-    (fp_line (start -3.3 -0.7) (end 3.3 -0.7) (layer B.SilkS) (width 0.001))
-    (fp_line (start 3.3 -0.7) (end 3.3 0) (layer B.SilkS) (width 0.001))
-    (fp_line (start -3.3 0) (end -3.3 6.8) (layer B.SilkS) (width 0.001))
-    (fp_line (start -3.3 6.8) (end 3.3 6.8) (layer B.SilkS) (width 0.001))
-    (fp_line (start 3.3 6.8) (end 3.3 0) (layer B.SilkS) (width 0.001))
-    (fp_line (start 3.3 0) (end -3.3 0) (layer B.SilkS) (width 0.001))
-    (pad 1 smd rect (at 1.8 6.475) (size 0.23 0.85) (layers B.Cu B.Paste B.Mask))
-    (pad 3 smd rect (at 1.4 6.475) (size 0.23 0.85) (layers B.Cu B.Paste B.Mask))
-    (pad 5 smd rect (at 1 6.475) (size 0.23 0.85) (layers B.Cu B.Paste B.Mask))
-    (pad 7 smd rect (at 0.6 6.475) (size 0.23 0.85) (layers B.Cu B.Paste B.Mask))
-    (pad 9 smd rect (at 0.2 6.475) (size 0.23 0.85) (layers B.Cu B.Paste B.Mask))
-    (pad 11 smd rect (at -0.2 6.475) (size 0.23 0.85) (layers B.Cu B.Paste B.Mask))
-    (pad 13 smd rect (at -0.6 6.475) (size 0.23 0.85) (layers B.Cu B.Paste B.Mask))
-    (pad 15 smd rect (at -1 6.475) (size 0.23 0.85) (layers B.Cu B.Paste B.Mask))
-    (pad 17 smd rect (at -1.4 6.475) (size 0.23 0.85) (layers B.Cu B.Paste B.Mask))
-    (pad 19 smd rect (at -1.8 6.475) (size 0.23 0.85) (layers B.Cu B.Paste B.Mask))
-    (pad 2 smd rect (at 1.6 5.25) (size 0.23 1) (layers B.Cu B.Paste B.Mask))
-    (pad 4 smd rect (at 1.2 5.25) (size 0.23 1) (layers B.Cu B.Paste B.Mask))
-    (pad 6 smd rect (at 0.8 5.25) (size 0.23 1) (layers B.Cu B.Paste B.Mask))
-    (pad 8 smd rect (at 0.4 5.25) (size 0.23 1) (layers B.Cu B.Paste B.Mask))
-    (pad 10 smd rect (at 0 5.25) (size 0.23 1) (layers B.Cu B.Paste B.Mask))
-    (pad 12 smd rect (at -0.4 5.25) (size 0.23 1) (layers B.Cu B.Paste B.Mask))
-    (pad 14 smd rect (at -0.8 5.25) (size 0.23 1) (layers B.Cu B.Paste B.Mask))
-    (pad 16 smd rect (at -1.2 5.25) (size 0.23 1) (layers B.Cu B.Paste B.Mask))
-    (pad 18 smd rect (at -1.6 5.25) (size 0.23 1) (layers B.Cu B.Paste B.Mask))
-    (pad SHD smd rect (at 3.45 5.06) (size 2.4 1.38) (layers B.Cu B.Paste B.Mask))
-    (pad SHD smd rect (at -3.45 5.06) (size 2.4 1.38) (layers B.Cu B.Paste B.Mask))
-    (pad "" thru_hole oval (at -3.1 1.7) (size 1.5 2.55) (drill oval 0.65 1.7) (layers *.Cu *.Mask B.SilkS))
-    (pad "" thru_hole oval (at 3.1 1.7) (size 1.5 2.55) (drill oval 0.65 1.7) (layers *.Cu *.Mask B.SilkS))
   )
   (module SMD_Packages:SSOP-20 (layer B.Cu)
@@
     )
   )
+  (module micro-hdmi-d:MICRO-HDMI-D (layer B.Cu)
+    (at 168.91 81.11)
+    (attr smd)
+    (fp_text reference P1 (at -0.025 3.125) (layer B.SilkS)
+      (effects (font (size 0.3 0.3) (thickness 0.075)) (justify mirror))
+    )
+    (fp_text value MICRO-HDMI-D (at 0 1.6) (layer B.SilkS)
+      (effects (font (size 0.3 0.3) (thickness 0.075)) (justify mirror))
+    )
+    (fp_line (start -3.3 0) (end -3.3 -0.7) (layer B.SilkS) (width 0.001))
+    (fp_line (start -3.3 -0.7) (end 3.3 -0.7) (layer B.SilkS) (width 0.001))
+    (fp_line (start 3.3 -0.7) (end 3.3 0) (layer B.SilkS) (width 0.001))
+    (fp_line (start -3.3 0) (end -3.3 6.8) (layer B.SilkS) (width 0.001))
+    (fp_line (start -3.3 6.8) (end 3.3 6.8) (layer B.SilkS) (width 0.001))
+    (fp_line (start 3.3 6.8) (end 3.3 0) (layer B.SilkS) (width 0.001))
+    (fp_line (start 3.3 0) (end -3.3 0) (layer B.SilkS) (width 0.001))
+    (pad 1 smd rect (at 1.8 6.475) (size 0.23 0.85) (layers B.Cu B.Paste B.Mask))
+    (pad 3 smd rect (at 1.4 6.475) (size 0.23 0.85) (layers B.Cu B.Paste B.Mask))
+    (pad 5 smd rect (at 1 6.475) (size 0.23 0.85) (layers B.Cu B.Paste B.Mask))
+    (pad 7 smd rect (at 0.6 6.475) (size 0.23 0.85) (layers B.Cu B.Paste B.Mask))
+    (pad 9 smd rect (at 0.2 6.475) (size 0.23 0.85) (layers B.Cu B.Paste B.Mask))
+    (pad 11 smd rect (at -0.2 6.475) (size 0.23 0.85) (layers B.Cu B.Paste B.Mask))
+    (pad 13 smd rect (at -0.6 6.475) (size 0.23 0.85) (layers B.Cu B.Paste B.Mask))
+    (pad 15 smd rect (at -1 6.475) (size 0.23 0.85) (layers B.Cu B.Paste B.Mask))
+    (pad 17 smd rect (at -1.4 6.475) (size 0.23 0.85) (layers B.Cu B.Paste B.Mask))
+    (pad 19 smd rect (at -1.8 6.475) (size 0.23 0.85) (layers B.Cu B.Paste B.Mask))
+    (pad 2 smd rect (at 1.6 5.25) (size 0.23 1) (layers B.Cu B.Paste B.Mask))
+    (pad 4 smd rect (at 1.2 5.25) (size 0.23 1) (layers B.Cu B.Paste B.Mask))
+    (pad 6 smd rect (at 0.8 5.25) (size 0.23 1) (layers B.Cu B.Paste B.Mask))
+    (pad 8 smd rect (at 0.4 5.25) (size 0.23 1) (layers B.Cu B.Paste B.Mask))
+    (pad 10 smd rect (at 0 5.25) (size 0.23 1) (layers B.Cu B.Paste B.Mask))
+    (pad 12 smd rect (at -0.4 5.25) (size 0.23 1) (layers B.Cu B.Paste B.Mask))
+    (pad 14 smd rect (at -0.8 5.25) (size 0.23 1) (layers B.Cu B.Paste B.Mask))
+    (pad 16 smd rect (at -1.2 5.25) (size 0.23 1) (layers B.Cu B.Paste B.Mask))
+    (pad 18 smd rect (at -1.6 5.25) (size 0.23 1) (layers B.Cu B.Paste B.Mask))
+    (pad 0 smd rect (at 3.45 5.06) (size 2.4 1.38) (layers B.Cu B.Paste B.Mask)
+      (net 13 "Net-(P1-Pad0)"))
+    (pad 0 smd rect (at -3.45 5.06) (size 2.4 1.38) (layers B.Cu B.Paste B.Mask)
+      (net 13 "Net-(P1-Pad0)"))
+    (pad "" thru_hole oval (at -3.1 1.7) (size 1.5 2.55) (drill oval 0.65 1.7) (layers *.Cu *.Mask B.SilkS))
+    (pad "" thru_hole oval (at 3.1 1.7) (size 1.5 2.55) (drill oval 0.65 1.7) (layers *.Cu *.Mask B.SilkS))
+  )
   (gr_line (start 140.97 81.28) (end 140.97 142.24) (layer Edge.Cuts) (width 0.15))
